File: left/left.kicad_pcb (KiCad board)
At the start: 2 copper layers, 53 parts, among them J1 MJ-4PP-9, U1 ProMicro

Commit message: PCBの外枠追加
Parts:
- added Ref**: Val**, kbd:HOLE, F.Cu at (207.0, 114.5)
- added Ref01: Val01, kbd:HOLE, F.Cu at (58.5, 32.0)
- added Ref02: Val02, kbd:HOLE, F.Cu at (207.0, 32.0)
- added Ref03: Val03, kbd:HOLE, F.Cu at (58.5, 81.5)
Other:
- board outline added: 158.5 x 116.8 mm
Changed lines of the file:
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@@
       (net 27 "Net-(D23-A)") (pinfunction "2") (pintype "passive"))
   )
+  (footprint "kbd:HOLE" (layer "F.Cu")
+    (at 58.5 81.5)
+    (descr "Mounting Hole 2.2mm, no annular, M2")
+    (tags "mounting hole 2.2mm no annular m2")
+    (attr exclude_from_pos_files exclude_from_bom)
+    (fp_text reference "Ref03" (at 0 -3.2) (layer "F.Fab")
+        (effects (font (size 1 1) (thickness 0.15)))
+    )
+    (fp_text value "Val03" (at 0 3.2) (layer "F.Fab")
+        (effects (font (size 1 1) (thickness 0.15)))
+    )
+    (fp_text user "${REFERENCE}" (at 0.3 0) (layer "F.Fab")
+        (effects (font (size 1 1) (thickness 0.15)))
+    )
+    (fp_circle (center 0 0) (end 2.2 0)
+      (stroke (width 0.15) (type solid)) (fill none) (layer "Cmts.User"))
+    (fp_circle (center 0 0) (end 2.45 0)
+      (stroke (width 0.05) (type solid)) (fill none) (layer "F.CrtYd"))
+    (pad "" np_thru_hole circle (at 0 0) (size 5 5) (drill 4.8) (layers "*.Cu" "*.Mask"))
+  )
   (footprint "kbd:D3_TH_SMD" (layer "F.Cu")
     (at 109 93.98)
@@
     )
   )
+  (footprint "kbd:HOLE" (layer "F.Cu")
+    (at 58.5 32)
+    (descr "Mounting Hole 2.2mm, no annular, M2")
+    (tags "mounting hole 2.2mm no annular m2")
+    (attr exclude_from_pos_files exclude_from_bom)
+    (fp_text reference "Ref01" (at 0 -3.2) (layer "F.Fab")
+        (effects (font (size 1 1) (thickness 0.15)))
+    )
+    (fp_text value "Val01" (at 0 3.2) (layer "F.Fab")
+        (effects (font (size 1 1) (thickness 0.15)))
+    )
+    (fp_text user "${REFERENCE}" (at 0.3 0) (layer "F.Fab")
+        (effects (font (size 1 1) (thickness 0.15)))
+    )
+    (fp_circle (center 0 0) (end 2.2 0)
+      (stroke (width 0.15) (type solid)) (fill none) (layer "Cmts.User"))
+    (fp_circle (center 0 0) (end 2.45 0)
+      (stroke (width 0.05) (type solid)) (fill none) (layer "F.CrtYd"))
+    (pad "" np_thru_hole circle (at 0 0) (size 5 5) (drill 4.8) (layers "*.Cu" "*.Mask"))
+  )
   (footprint "kbd:CherryMX_Choc_Hotswap" (layer "F.Cu")
     (at 200.5 132.98)
@@
       (net 21 "Net-(D18-A)") (pinfunction "2") (pintype "passive"))
   )
+  (footprint "kbd:HOLE" (layer "F.Cu")
+    (at 207 32)
+    (descr "Mounting Hole 2.2mm, no annular, M2")
+    (tags "mounting hole 2.2mm no annular m2")
+    (attr exclude_from_pos_files exclude_from_bom)
+    (fp_text reference "Ref02" (at 0 -3.2) (layer "F.Fab")
+        (effects (font (size 1 1) (thickness 0.15)))
+    )
+    (fp_text value "Val02" (at 0 3.2) (layer "F.Fab")
+        (effects (font (size 1 1) (thickness 0.15)))
+    )
+    (fp_text user "${REFERENCE}" (at 0.3 0) (layer "F.Fab")
+        (effects (font (size 1 1) (thickness 0.15)))
+    )
+    (fp_circle (center 0 0) (end 2.2 0)
+      (stroke (width 0.15) (type solid)) (fill none) (layer "Cmts.User"))
+    (fp_circle (center 0 0) (end 2.45 0)
+      (stroke (width 0.05) (type solid)) (fill none) (layer "F.CrtYd"))
+    (pad "" np_thru_hole circle (at 0 0) (size 5 5) (drill 4.8) (layers "*.Cu" "*.Mask"))
+  )
   (footprint "kbd:CherryMX_Choc_Hotswap" (layer "F.Cu")
     (at 95.5 42.98)
@@
       (net 7 "Net-(D6-A)") (pinfunction "2") (pintype "passive"))
   )
+  (footprint "kbd:HOLE" (layer "F.Cu")
+    (at 207 114.5)
+    (descr "Mounting Hole 2.2mm, no annular, M2")
+    (tags "mounting hole 2.2mm no annular m2")
+    (attr exclude_from_pos_files exclude_from_bom)
+    (fp_text reference "Ref**" (at 0 -3.2) (layer "F.Fab")
+        (effects (font (size 1 1) (thickness 0.15)))
+    )
+    (fp_text value "Val**" (at 0 3.2) (layer "F.Fab")
+        (effects (font (size 1 1) (thickness 0.15)))
+    )
+    (fp_text user "${REFERENCE}" (at 0.3 0) (layer "F.Fab")
+        (effects (font (size 1 1) (thickness 0.15)))
+    )
+    (fp_circle (center 0 0) (end 2.2 0)
+      (stroke (width 0.15) (type solid)) (fill none) (layer "Cmts.User"))
+    (fp_circle (center 0 0) (end 2.45 0)
+      (stroke (width 0.05) (type solid)) (fill none) (layer "F.CrtYd"))
+    (pad "" np_thru_hole circle (at 0 0) (size 5 5) (drill 4.8) (layers "*.Cu" "*.Mask"))
+  )
   (footprint "kbd:CherryMX_Choc_Hotswap" (layer "F.Cu")
     (at 109 82.98)
@@
     )
   )
+  (gr_line (start 53.5 118) (end 53.5 28)
+    (stroke (width 0.1) (type default)) (layer "Edge.Cuts"))
+  (gr_line (start 212 28) (end 212 144.78)
+    (stroke (width 0.1) (type default)) (layer "Edge.Cuts"))
+  (gr_line (start 212 144.78) (end 187.96 144.78)
+    (stroke (width 0.1) (type default)) (layer "Edge.Cuts"))
+  (gr_line (start 175.26 118) (end 187.96 144.78)
+    (stroke (width 0.1) (type default)) (layer "Edge.Cuts"))
+  (gr_line (start 53.5 118) (end 175.26 118)
+    (stroke (width 0.1) (type default)) (layer "Edge.Cuts"))
+  (gr_line (start 53.5 28) (end 212 28)
+    (stroke (width 0.1) (type default)) (layer "Edge.Cuts"))
 )
