File: left/left.kicad_sch (KiCad schematic)
At the start: 55 parts, among them J1 MJ-4PP-9, U1 ProMicro

Commit message: updated PCB
Parts:
- removed D19: D, kbd:D3_TH_SMD, symbol Device:D
- removed LEFT_SW19: SW_PUSH, kbd:CherryMX_Choc_Hotswap, symbol kbd:SW_PUSH
- LEFT_SW13, LEFT_SW7: footprint kbd:CherryMX_Choc_Hotswap -> kbd:CherryMX_Choc_Hotswap_1.5u
- renumbered D20 to D19, D21 to D20, D22 to D21, D23 to D22, D24 to D23, D25 to D24, D26 to D25, LEFT_SW20 to LEFT_SW19, LEFT_SW21 to LEFT_SW20, LEFT_SW22 to LEFT_SW21, LEFT_SW23 to LEFT_SW22, LEFT_SW24 to LEFT_SW23, LEFT_SW25 to LEFT_SW24, LEFT_SW26 to LEFT_SW25

Commit message: 左手PCBの組み換え．外枠は未完成
Parts:
- removed D25: D, kbd:D3_TH_SMD, symbol Device:D
- removed LEFT_SW25: SW_PUSH, kbd:CherryMX_Choc_Hotswap, symbol kbd:SW_PUSH
- LEFT_SW13, LEFT_SW22, LEFT_SW7: footprint kbd:CherryMX_Choc_Hotswap_1.5u -> kbd:CherryMX_Choc_Hotswap
- LEFT_SW15: footprint kbd:CherryMX_Choc_Hotswap -> kbd:CherryMX_Choc_Hotswap_1.5u
Connections:
- net col1: now also LEFT_SW15.1, LEFT_SW8.1; no longer LEFT_SW13.1, LEFT_SW7.1
- net col2: now also LEFT_SW16.1, LEFT_SW9.1; no longer LEFT_SW14.1, LEFT_SW19.1, LEFT_SW8.1
- net col3: now also LEFT_SW10.1, LEFT_SW17.1; no longer LEFT_SW15.1, LEFT_SW20.1, LEFT_SW9.1
- net col4: now also LEFT_SW11.1, LEFT_SW18.1; no longer LEFT_SW10.1, LEFT_SW16.1
- net col5: now also LEFT_SW12.1, LEFT_SW19.1; no longer LEFT_SW11.1, LEFT_SW17.1
- net col6: now also LEFT_SW13.1, LEFT_SW20.1; no longer LEFT_SW12.1, LEFT_SW18.1
- net col7: now also LEFT_SW14.1, LEFT_SW7.1
- net row1: now also D7.1 (K); no longer D24.1 (K)
- net row2: now also D13.1 (K), D14.1 (K); no longer D7.1 (K)
- net row3: now also D19.1 (K), D20.1 (K); no longer D13.1 (K), D14.1 (K)
- net row4: now also D24.1 (K); no longer D19.1 (K), D20.1 (K)
