File: right/right.kicad_sch (KiCad schematic)
At the start: 55 parts, among them J1 MJ-4PP-9, U1 ProMicro_r

Commit message: 右手PCB作成
Parts:
- RIGHT_SW13, RIGHT_SW26, RIGHT_SW6: footprint kbd:CherryMX_Choc_Hotswap -> kbd:CherryMX_Choc_Hotswap_1.5u
Connections:
- net col1: now also RIGHT_SW14.1, RIGHT_SW8.1
- net col2: now also RIGHT_SW15.1, RIGHT_SW9.1; no longer RIGHT_SW14.1, RIGHT_SW8.1
- net col3: now also RIGHT_SW10.1, RIGHT_SW16.1; no longer RIGHT_SW15.1, RIGHT_SW9.1
- net col4: now also RIGHT_SW11.1, RIGHT_SW17.1; no longer RIGHT_SW10.1, RIGHT_SW16.1
- net col5: now also RIGHT_SW12.1, RIGHT_SW18.1; no longer RIGHT_SW11.1, RIGHT_SW17.1
- net col6: now also RIGHT_SW13.1, RIGHT_SW19.1; no longer RIGHT_SW12.1, RIGHT_SW18.1
- net col7: no longer RIGHT_SW13.1, RIGHT_SW19.1
Other:
- moved on the sheet: D10, D11, D12, D13, D14, D15, D16, D17, D18, D19, D8, D9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
