File: v1.0/v1.0.kicad_sch (KiCad schematic)
At the start: 41 parts, among them J1 MJ-4PP-9, SW1 SW_PUSH, SW10 SW_PUSH, SW11 SW_PUSH, SW12 SW_PUSH, SW13 SW_PUSH, SW14 SW_PUSH, SW15 SW_PUSH, SW16 SW_PUSH, SW17 SW_PUSH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

Commit message: updated
Parts:
- added U2: switch, otborad:triangle, symbol ot_board:switch
- added U3: RKJXV122400R, otborad:RKJXV122400R, symbol ot_board:RKJXV122400R
- J1: footprint kbd:MJ-4PP-9 -> otborad:MJ-4PP-9_reversible
- SW1, SW10, SW11, SW12, SW13, SW14, SW15, SW16, SW17, SW18, SW19, SW2, SW3, SW4, SW5, SW6, SW7, SW8, SW9: footprint footprint:keyswitch_choc12_hotswap_1u_rev -> otborad:choc1_0.8u_reversible
- U1: footprint footprint:ProMicro -> otborad:ProMicro
Connections:
- net GND: now also U2.2 (GND), U3.1 (GND)
- net VCC: now also U2.1 (VCC), U3.3 (VCC); no longer U1.2 (RX1/D2)
- net row1: now also U1.7 (4/D4); no longer U1.9 (6/D7)
- net row2: now also U1.9 (6/D7); no longer U1.10 (7/E6)
- net row3: now also U1.10 (7/E6); no longer U1.11 (8/B4)
- net row4: now also U1.20 (F4/A3); no longer U1.12 (9/B5)
- new net VRx: U1.11 (8/B4), U3.2 (VRx)
- new net VRy: U1.12 (9/B5), U3.4 (VRy)
- new net switch: U1.2 (RX1/D2), U2.3 (switch)
- no-connect marks 7 -> 9

Commit message: updated
Parts:
- added D20: D, Keebio-Parts:Diode-dual, symbol Device:D
- added SW21: SW_PUSH, kbd:ResetSW, symbol kbd:SW_PUSH
- SW20: footprint kbd:ResetSW -> otborad:choc1_0.8u_reversible_uponly
Connections:
- net GND: now also SW21.2; no longer SW20.2
- net col4: now also SW20.1
- net reset: now also SW21.1; no longer SW20.1
- net row4: now also D20.1 (K)
- new net: D20.2 (A), SW20.2
Other:
- moved on the sheet: SW20
Changed lines of the file:
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@@
 	)
 	(junction
+		(at 163.83 115.57)
+		(diameter 0)
+		(color 0 0 0 0)
+	)
+	(junction
 		(at 186.69 93.98)
 		(diameter 0)
@@
 		(color 0 0 0 0)
 	)
+	(junction
+		(at 171.45 85.09)
+		(diameter 0)
+		(color 0 0 0 0)
+	)
 	(no_connect
 		(at 41.91 60.96)
@@
 	(wire
 		(pts
+			(xy 163.83 115.57) (xy 186.69 115.57)
+		)
+		(stroke
+			(width 0)
+			(type default)
+		)
+	)
+	(wire
+		(pts
 			(xy 232.41 41.91) (xy 232.41 43.18)
 		)
@@
 	(wire
 		(pts
+			(xy 171.45 85.09) (xy 171.45 105.41)
+		)
+		(stroke
+			(width 0)
+			(type default)
+		)
+	)
+	(wire
+		(pts
 			(xy 256.54 63.5) (xy 256.54 64.77)
 		)
@@
 	(wire
 		(pts
-			(xy 46.99 24.13) (xy 49.53 24.13)
-		)
-		(stroke
-			(width 0)
-			(type default)
-		)
-	)
-	(wire
-		(pts
 			(xy 29.21 88.9) (xy 30.48 88.9)
 		)
@@
 	(wire
 		(pts
+			(xy 64.77 24.13) (xy 64.77 25.4)
+		)
+		(stroke
+			(width 0)
+			(type default)
+		)
+	)
+	(wire
+		(pts
 			(xy 20.32 39.37) (xy 24.13 39.37)
 		)
@@
 	(wire
 		(pts
+			(xy 46.99 24.13) (xy 49.53 24.13)
+		)
+		(stroke
+			(width 0)
+			(type default)
+		)
+	)
+	(wire
+		(pts
 			(xy 140.97 72.39) (xy 163.83 72.39)
 		)
@@
 	(wire
 		(pts
-			(xy 64.77 24.13) (xy 64.77 25.4)
+			(xy 186.69 105.41) (xy 186.69 107.95)
 		)
 		(stroke
@@
 	(symbol
 		(lib_id "kbd:SW_PUSH")
-		(at 57.15 24.13 0)
+		(at 179.07 105.41 0)
 		(unit 1)
 		(exclude_from_sim no)
@@
 		(fields_autoplaced yes)
 		(property "Reference" "SW20"
-			(at 57.15 16.51 0)
+			(at 179.07 97.79 0)
 			(effects
 				(font
@@
 		)
 		(property "Value" "SW_PUSH"
-			(at 57.15 19.05 0)
+			(at 179.07 100.33 0)
 			(effects
 				(font
@@
 			)
 		)
-		(property "Footprint" "kbd:ResetSW"
-			(at 57.15 24.13 0)
+		(property "Footprint" "otborad:choc1_0.8u_reversible_uponly"
+			(at 179.07 105.41 0)
 			(effects
 				(font
@@
 		)
 		(property "Datasheet" ""
-			(at 57.15 24.13 0)
+			(at 179.07 105.41 0)
 			(effects
 				(font
@@
 		)
 		(property "Description" ""
-			(at 57.15 24.13 0)
+			(at 179.07 105.41 0)
 			(effects
 				(font
@@
 	(symbol
 		(lib_id "Device:D")
+		(at 186.69 111.76 90)
+		(unit 1)
+		(exclude_from_sim no)
+		(in_bom yes)
+		(on_board yes)
+		(dnp no)
+		(fields_autoplaced yes)
+		(property "Reference" "D20"
+			(at 189.23 110.4899 90)
+			(effects
+				(font
+					(size 1.27 1.27)
+				)
+				(justify right)
+			)
+		)
+		(property "Value" "D"
+			(at 189.23 113.0299 90)
+			(effects
+				(font
+					(size 1.27 1.27)
+				)
+				(justify right)
+			)
+		)
+		(property "Footprint" "Keebio-Parts:Diode-dual"
+			(at 186.69 111.76 0)
+			(effects
+				(font
+					(size 1.27 1.27)
+				)
+				(hide yes)
+			)
+		)
+		(property "Datasheet" "~"
+			(at 186.69 111.76 0)
+			(effects
+				(font
+					(size 1.27 1.27)
+				)
+				(hide yes)
+			)
+		)
+		(property "Description" "Diode"
+			(at 186.69 111.76 0)
+			(effects
+				(font
+					(size 1.27 1.27)
+				)
+				(hide yes)
+			)
+		)
+		(property "Sim.Device" "D"
+			(at 186.69 111.76 0)
+			(effects
+				(font
+					(size 1.27 1.27)
+				)
+				(hide yes)
+			)
+		)
+		(property "Sim.Pins" "1=K 2=A"
+			(at 186.69 111.76 0)
+			(effects
+				(font
+					(size 1.27 1.27)
+				)
+				(hide yes)
+			)
+		)
+		(pin "2"
+		)
+		(pin "1"
+		)
+		(instances
+			(project ""
+				(path "/df4eae37-4127-470e-becc-662440e2186b"
+					(reference "D20")
+					(unit 1)
+				)
+			)
+		)
+	)
+	(symbol
+		(lib_id "Device:D")
 		(at 186.69 46.99 90)
 		(unit 1)
@@
 					(unit 1)
 				)
+			)
+		)
+	)
+	(symbol
+		(lib_id "kbd:SW_PUSH")
+		(at 57.15 24.13 0)
+		(unit 1)
+		(exclude_from_sim no)
+		(in_bom yes)
+		(on_board yes)
+		(dnp no)
+		(fields_autoplaced yes)
+		(property "Reference" "SW21"
+			(at 57.15 16.51 0)
+			(effects
+				(font
+					(size 1.27 1.27)
+				)
+			)
+		)
+		(property "Value" "SW_PUSH"
+			(at 57.15 19.05 0)
+			(effects
+				(font
+					(size 1.27 1.27)
+				)
+			)
+		)
+		(property "Footprint" "kbd:ResetSW"
+			(at 57.15 24.13 0)
+			(effects
+				(font
+					(size 1.27 1.27)
+				)
+				(hide yes)
+			)
+		)
+		(property "Datasheet" ""
+			(at 57.15 24.13 0)
+			(effects
+				(font
+					(size 1.27 1.27)
+				)
+			)
+		)
+		(property "Description" ""
+			(at 57.15 24.13 0)
+			(effects
+				(font
+					(size 1.27 1.27)
+				)
+				(hide yes)
+			)
+		)
+		(pin "1"
+		)
+		(pin "2"
+		)
+		(instances
+			(project ""
+				(path "/df4eae37-4127-470e-becc-662440e2186b"
+					(reference "SW21")
+					(unit 1)
+				)
