File: v2.0/v2.0.kicad_sch (KiCad schematic)
At the start: 46 parts, among them J1 MJ-4PP-9, SW1 SW_PUSH, SW10 SW_PUSH, SW11 SW_PUSH, SW12 SW_PUSH, SW13 SW_PUSH, SW14 SW_PUSH, SW15 SW_PUSH, SW16 SW_PUSH, SW17 SW_PUSH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

Commit message: updated
Parts:
- added D22, D23, D24: D, Keebio-Parts:Diode-dual, symbol Device:D
- added SW23, SW24: SW_PUSH, otborad:choc1_0.8u_reversible, symbol kbd:SW_PUSH
- added SW25: SW_PUSH, kbd:ResetSW, symbol kbd:SW_PUSH
- SW22: footprint kbd:ResetSW -> otborad:choc1_0.8u_reversible
Connections:
- net GND: now also SW25.2; no longer SW22.2
- net col1: now also SW13.1, SW19.1, SW7.1; no longer SW12.1, SW18.1, SW6.1
- net col2: now also SW14.1, SW20.1, SW8.1; no longer SW13.1, SW19.1, SW7.1
- net col3: now also SW15.1, SW21.1, SW9.1; no longer SW14.1, SW20.1, SW8.1
- net col4: now also SW10.1, SW16.1, SW22.1; no longer SW15.1, SW21.1, SW9.1
- net col5: now also SW11.1, SW17.1, SW23.1; no longer SW10.1, SW16.1
- net col6: now also SW12.1, SW18.1, SW6.1, SW24.1; no longer SW11.1, SW17.1
- net reset: now also SW25.1; no longer SW22.1
- net row1: now also D6.1 (K)
- net row2: now also D12.1 (K); no longer D6.1 (K)
- net row3: now also D18.1 (K); no longer D12.1 (K)
- net row4: now also D22.1 (K), D23.1 (K), D24.1 (K); no longer D18.1 (K)
- new net: D24.2 (A), SW24.2
- new net: D22.2 (A), SW22.2
- new net: D23.2 (A), SW23.2
Other:
- moved on the sheet: D10, D11, D12, D13, D14, D15, D16, D17, D18, D19, D20, D21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
